Commit message: add second laser, extend FOV, and reposition higher

File: robots/youbot_base_only.urdf.xacro (robot description, xacro)
@@ -27,6 +27,10 @@
   <xacro:youbot_base name="base"/>
   <!-- base laser front -->
-  <xacro:hokuyo_urg04_laser name="base_laser_front" parent="base" ros_topic="scan" update_rate="50" min_angle="-1.57" max_angle="1.57">
-    <origin xyz="0.3 0 -0.03" rpy="0 0 0"/>
+  <xacro:hokuyo_urg04_laser name="base_laser_front" parent="base" ros_topic="scan_1" update_rate="40" min_angle="-2.36" max_angle="2.36">
+    <origin xyz="0.3 0 0.04" rpy="0 0 0"/>
+  </xacro:hokuyo_urg04_laser>
+  <!-- base laser back -->
+  <xacro:hokuyo_urg04_laser name="base_laser_back" parent="base" ros_topic="scan_2" update_rate="40" min_angle="-2.36" max_angle="2.36">
+    <origin xyz="-0.3 0 0.04" rpy="0 0 3.1415"/>
   </xacro:hokuyo_urg04_laser>
 </robot>
