Commit message: Modified URDF so depth cam sits on gripper.

File: robots/youbot_with_cam3d.urdf.xacro (robot description, xacro)
@@ -23,6 +23,4 @@
   <xacro:include filename="$(find youbot_description)/urdf/sensors/hokuyo_urg04_laser.urdf.xacro"/>
   <xacro:include filename="$(find youbot_description)/urdf/sensors/asus_xtion_camera.urdf.xacro"/>
-  <!-- sensor tower -->
-  <xacro:include filename="$(find youbot_description)/urdf/misc/camera_tower.urdf.xacro"/>
   <!-- Now we can start using the macros xacro:included above to define the actual youbot -->
   <!-- The first use of a macro.  This one was defined in base.urdf.xacro above.
@@ -48,11 +46,7 @@
     <origin xyz="0.3 0 -0.03" rpy="0 0 0"/>
   </xacro:hokuyo_urg04_laser>
-  <!-- camera tower -->
-  <xacro:camera_tower name="camera_tower" parent="plate_link">
-    <origin xyz="-0.11 0.0 0.03" rpy="0 0 0" />
-  </xacro:camera_tower>
-  <!-- 3D camera on tower -->
-  <xacro:asus_xtion_camera name="tower_cam3d" parent="camera_tower_link" tilt="0.5">
-    <origin xyz="0 0 0.49" rpy="0 0 0" />
+  <!-- 3D camera on gripper -->
+  <xacro:asus_xtion_camera name="tower_cam3d" parent="gripper_palm_link" tilt="0.0">
+    <origin xyz="-0.02 0 -0.035" rpy="0 -1.5 0" />
   </xacro:asus_xtion_camera>
 </robot>

Commit message: Mouted camera on the correct side of the gripper now.

File: robots/youbot_with_cam3d.urdf.xacro (robot description, xacro)
@@ -47,6 +47,6 @@
   </xacro:hokuyo_urg04_laser>
   <!-- 3D camera on gripper -->
-  <xacro:asus_xtion_camera name="tower_cam3d" parent="gripper_palm_link" tilt="0.0">
-    <origin xyz="-0.02 0 -0.035" rpy="0 -1.5 0" />
+  <xacro:asus_xtion_camera name="depth_cam" parent="gripper_palm_link" tilt="0.0">
+    <origin xyz="0.025 0 -0.035" rpy="${M_PI} -${M_PI/2} 0" />
   </xacro:asus_xtion_camera>
 </robot>

Commit message: Modified Friction fro link 1 2 3. mounted cam on right side now.

File: robots/youbot_with_cam3d.urdf.xacro (robot description, xacro)
@@ -48,5 +48,5 @@
   <!-- 3D camera on gripper -->
   <xacro:asus_xtion_camera name="depth_cam" parent="gripper_palm_link" tilt="0.0">
-    <origin xyz="0.025 0 -0.035" rpy="${M_PI} -${M_PI/2} 0" />
+    <origin xyz="-0.02 0 -0.035" rpy="0 -1.5 0" />
   </xacro:asus_xtion_camera>
 </robot>

File: urdf/youbot_arm/arm.urdf.xacro (robot description, xacro)
@@ -44,5 +44,5 @@
 			<axis xyz="0 0 -1"/>
 			<!--<calibration rising="${arm_1_ref}" falling="${arm_1_ref}"/>-->
-			<dynamics damping="1" friction="1" />
+			<dynamics damping="1" friction="0.5" />
 			<!-- damping - N*s/m, N*s*m/rad -->
 			<!-- friction - N, N*m -->
@@ -83,5 +83,5 @@
 			<axis xyz="0 1 0"/>
 			<!--<calibration rising="${arm_2_ref}" falling="${arm_2_ref}"/>-->
-			<dynamics damping="1" friction="1" />
+			<dynamics damping="1" friction="0.5" />
 			<limit effort="${9.5}" velocity="${M_PI / 2.0}" lower="0" upper="${joint_2_limit}"/>
       <!--safety_controller k_position="20" k_velocity="${2*9.5/M_PI}" soft_lower_limit="${threshold}" soft_upper_limit="${joint_2_limit_soft}" /-->
@@ -122,5 +122,5 @@
 			<child link="${name}_link_3"/>
 			<axis xyz="0 1 0"/>
-			<dynamics damping="1" friction="1" />
+			<dynamics damping="1" friction="0.5" />
 			<limit effort="${6.0}" velocity="${M_PI / 2.0}" lower="-${joint_3_limit}" upper="0"/>
       <!--safety_controller k_position="20" k_velocity="50" soft_lower_limit="-${joint_3_limit_soft}" soft_upper_limit="-${threshold}" /-->

File: urdf/youbot_gripper/gripper.urdf.xacro (robot description, xacro)
@@ -40,5 +40,5 @@
 			<child link="${name}_finger_link_l"/>
 			<axis xyz="0 -1 0" />
-			<dynamics damping="1.0" friction="1.0" />
+			<dynamics damping="1.0" friction="0.5" />
 			<limit effort="1" velocity="0.1" lower="0" upper="${finger_joint}"/>
                         <safety_controller k_position="20" k_velocity="25" soft_lower_limit="${threshold}" soft_upper_limit="${finger_joint_soft}" />
@@ -70,5 +70,5 @@
 			<child link="${name}_finger_link_r"/>
 			<axis xyz="0 -1 0" />
-			<dynamics damping="1.0" friction="1.0" />
+			<dynamics damping="1.0" friction="0.5" />
 			<limit effort="1" velocity="0.1" lower="0" upper="${finger_joint}"/>
                         <safety_controller k_position="20" k_velocity="25" soft_lower_limit="${threshold}" soft_upper_limit="${finger_joint_soft}" />
