Commit message: reposition IMU to the center

File: urdf/sensors/imu.urdf.xacro (robot description, xacro)
@@ -3,5 +3,5 @@
 <robot name="youbot_base_only" xmlns:xacro="http://www.ros.org/wiki/xacro">
   <!-- Constants for robot dimensions -->
-  <xacro:property name="height" value="0.046" /> <!-- Link X -->
+  <xacro:property name="height" value="0.04" /> <!-- Link X -->
   <xacro:property name="imu_link" value="0.05" /> <!-- Size of square 'IMU' box -->
   <!-- Import all Gazebo-customization elements, including Gazebo colors -->
@@ -12,5 +12,5 @@
   <joint name="imu_joint" type="fixed">
     <axis xyz="0 1 0" />
-    <origin xyz="${imu_link} 0 ${height}" rpy="0 0 0"/>
+    <origin xyz="0 0 ${height}" rpy="0 0 0"/>
     <parent link="base_link"/>
     <child link="imu_link"/>

Commit message: fix IMU joint

File: urdf/sensors/imu.urdf.xacro (robot description, xacro)
@@ -11,5 +11,5 @@
   <!-- IMU joint -->
   <joint name="imu_joint" type="fixed">
-    <axis xyz="0 1 0" />
+    <axis xyz="0 0 0" />
     <origin xyz="0 0 ${height}" rpy="0 0 0"/>
     <parent link="base_link"/>
