Commit message: Added D435 Mount.

File: urdf/sensors/intel_d435.urdf.xacro (robot description, xacro)
@@ -30,11 +30,64 @@
   </material>
   <xacro:macro name="intel_d435" params="name parent *origin tilt">
-    <!-- camera body, with origin at bottom screw mount -->
-    <joint name="camera_joint" type="fixed">
+    <link name="${name}_foot_link">
+      <inertial>
+        <mass value="0.05" />
+        <origin xyz="0 0 0" rpy="0 0 0"/>
+        <inertia ixx="0.0001" ixy="0" ixz="0" iyy="0.0001" iyz="0" izz="0.0001" />
+      </inertial>
+      <visual>
+        <origin xyz="0 0 0" rpy="${M_PI/2} 0 ${M_PI/2}" />
+        <geometry>
+          <mesh filename="package://youbot_description/meshes/sensors/d435_mount.dae"/>
+        </geometry>
+        <material name="Black" />
+      </visual>
+      <collision>
+        <origin xyz="0 0 0" rpy="${M_PI/2} 0 ${M_PI/2}" />
+        <geometry>
+          <mesh filename="package://youbot_description/meshes/sensors/d435_mount.dae"/>
+        </geometry>
+      </collision >
+    </link>
+    <joint name="${name}_foot_joint" type="fixed">
       <xacro:insert_block name="origin" />
       <parent link="${parent}"/>
-      <child link="camera_link" />
+      <child link="${name}_foot_link"/>
     </joint>
-    <link name="camera_link">
+    <link name="${name}_tilt_link">
+      <inertial>
+        <mass value="0.01" />
+        <origin xyz="0 0 0" rpy="0 0 0"/>
+        <inertia ixx="0.0001" ixy="0" ixz="0" iyy="0.0001" iyz="0" izz="0.0001" />
+      </inertial>
+      <visual>
+        <origin xyz="0 0 0.0075" rpy="0 0 0" />
+        <geometry>
+          <cylinder length="0.05" radius="0.003" />
+        </geometry>
+        <material name="aluminum"/>
+      </visual>
+      <collision>
+        <origin xyz="0 0 0.0075" rpy="0 0 0" />
+        <geometry>
+          <cylinder length="0.05" radius="0.003" />
+        </geometry>
+        <material name="aluminum"/>
+      </collision >
+    </link>
+    <joint name="intel_d435_tilt_joint" type="fixed">
+      <parent link="${name}_foot_link"/>
+      <child link="${name}_tilt_link"/>
+      <!--<axis xyz="0 1 0"/>-->
+      <origin xyz="0 0 0.0075" rpy="0 ${tilt} 0"/>
+      <!--<limit effort="100" lower="-0.541052068" upper="0.541052068" velocity="1.0"/>-->
+    </joint>
+    <!-- camera body, with origin at bottom screw mount -->
+    <joint name="${name}_camera_joint" type="fixed">
+      <origin xyz="0 0 0.03" rpy="0 0 0" />
+      <parent link="${name}_tilt_link"/>
+      <child link="${name}_camera" />
+    </joint>
+    <link name="${name}_camera">
       <visual>
       <origin xyz="${d435_cam_mount_from_center_offset} 0.0 ${d435_cam_height/2}" rpy="${M_PI/2} 0 ${M_PI/2}"/>
@@ -59,55 +112,55 @@
     </link>
     <!-- camera depth joints and links -->
-    <joint name="camera_depth_joint" type="fixed">
+    <joint name="${name}_depth_joint" type="fixed">
       <origin xyz="${d435_cam_depth_px} ${d435_cam_depth_py} ${d435_cam_depth_pz}" rpy="0 0 0"/>
-      <parent link="camera_link"/>
-      <child link="camera_depth_frame" />
+      <parent link="${name}_camera"/>
+      <child link="${name}_depth_frame" />
     </joint>
-    <link name="camera_depth_frame"/>
-    <joint name="camera_depth_optical_joint" type="fixed">
+    <link name="${name}_depth_frame"/>
+    <joint name="${name}_depth_optical_joint" type="fixed">
       <origin xyz="0 0 0" rpy="${-M_PI/2} 0 ${-M_PI/2}" />
-      <parent link="camera_depth_frame" />
-      <child link="camera_depth_optical_frame" />
+      <parent link="${name}_depth_frame" />
+      <child link="${name}_depth_optical_frame" />
     </joint>
-    <link name="camera_depth_optical_frame"/>
+    <link name="${name}_depth_optical_frame"/>
     <!-- camera left IR joints and links -->
-    <joint name="camera_left_ir_joint" type="fixed">
+    <joint name="${name}_left_ir_joint" type="fixed">
       <origin xyz="0 ${d435_cam_depth_to_left_ir_offset} 0" rpy="0 0 0" />
-      <parent link="camera_depth_frame" />
-      <child link="camera_left_ir_frame" />
+      <parent link="${name}_depth_frame" />
+      <child link="${name}_left_ir_frame" />
     </joint>
-    <link name="camera_left_ir_frame"/>
-    <joint name="camera_left_ir_optical_joint" type="fixed">
+    <link name="${name}_left_ir_frame"/>
+    <joint name="${name}_left_ir_optical_joint" type="fixed">
       <origin xyz="0 0 0" rpy="${-M_PI/2} 0 ${-M_PI/2}" />
-      <parent link="camera_left_ir_frame" />
-      <child link="camera_left_ir_optical_frame" />
+      <parent link="${name}_left_ir_frame" />
+      <child link="${name}_left_ir_optical_frame" />
     </joint>
-    <link name="camera_left_ir_optical_frame"/>
+    <link name="${name}_left_ir_optical_frame"/>
     <!-- camera right IR joints and links -->
-    <joint name="camera_right_ir_joint" type="fixed">
+    <joint name="${name}_right_ir_joint" type="fixed">
       <origin xyz="0 ${d435_cam_depth_to_right_ir_offset} 0" rpy="0 0 0" />
-      <parent link="camera_depth_frame" />
-      <child link="camera_right_ir_frame" />
+      <parent link="${name}_depth_frame" />
+      <child link="${name}_right_ir_frame" />
     </joint>
-    <link name="camera_right_ir_frame"/>
-    <joint name="camera_right_ir_optical_joint" type="fixed">
+    <link name="${name}_right_ir_frame"/>
+    <joint name="${name}_right_ir_optical_joint" type="fixed">
       <origin xyz="0 0 0" rpy="${-M_PI/2} 0 ${-M_PI/2}" />
-      <parent link="camera_right_ir_frame" />
-      <child link="camera_right_ir_optical_frame" />
+      <parent link="${name}_right_ir_frame" />
+      <child link="${name}_right_ir_optical_frame" />
     </joint>
-    <link name="camera_right_ir_optical_frame"/>
+    <link name="${name}_right_ir_optical_frame"/>
     <!-- camera fisheye joints and links -->
-    <joint name="camera_fisheye_joint" type="fixed">
+    <joint name="${name}_fisheye_joint" type="fixed">
       <origin xyz="0 ${d435_cam_depth_to_fisheye_offset} 0" rpy="0 0 0" />
-      <parent link="camera_depth_frame" />
-      <child link="camera_fisheye_frame" />
+      <parent link="${name}_depth_frame" />
+      <child link="${name}_fisheye_frame" />
     </joint>
-    <link name="camera_fisheye_frame"/>
-    <joint name="camera_fisheye_optical_joint" type="fixed">
+    <link name="${name}_fisheye_frame"/>
+    <joint name="${name}_fisheye_optical_joint" type="fixed">
       <origin xyz="0 0 0" rpy="${-M_PI/2} 0 ${-M_PI/2}" />
-      <parent link="camera_fisheye_frame" />
-      <child link="camera_fisheye_optical_frame" />
+      <parent link="${name}_fisheye_frame" />
+      <child link="${name}_fisheye_optical_frame" />
     </joint>
-    <link name="camera_fisheye_optical_frame"/>
+    <link name="${name}_fisheye_optical_frame"/>
     <xacro:intel_d435_gazebo name="${name}" />
   </xacro:macro>
