Commit message: Removed casters and added real youbot wheels. New movement plugin.

File: urdf/sensors/intel_d435.gazebo.xacro (robot description, xacro)
@@ -9,5 +9,5 @@
       <sensor type="depth" name="${name}_depth_frame_sensor">
         <always_on>true</always_on>
-        <update_rate>20.0</update_rate>
+        <update_rate>30.0</update_rate>
         <camera>
           <horizontal_fov>${87.0*M_PI/180.0}</horizontal_fov>
@@ -25,5 +25,5 @@
           <baseline>0.2</baseline>
           <alwaysOn>true</alwaysOn>
-          <updateRate>20.0</updateRate>
+          <updateRate>30.0</updateRate>
           <cameraName>${name}_depth</cameraName>
           <imageTopicName>/${name}/ir/image_raw</imageTopicName>
@@ -48,5 +48,5 @@
       <sensor type="depth" name="${name}_rgb_frame_sensor">
         <always_on>true</always_on>
-        <update_rate>20.0</update_rate>
+        <update_rate>30.0</update_rate>
         <camera>
           <horizontal_fov>${87.0*M_PI/180.0}</horizontal_fov>
@@ -64,5 +64,5 @@
           <baseline>0.2</baseline>
           <alwaysOn>true</alwaysOn>
-          <updateRate>20.0</updateRate>
+          <updateRate>30.0</updateRate>
           <cameraName>${name}_rgb</cameraName>
           <imageTopicName>/${name}/rgb/image_raw</imageTopicName>

File: urdf/youbot_base/base.gazebo.xacro (robot description, xacro)
@@ -4,5 +4,5 @@
        xmlns:interface="http://playerstage.sourceforge.net/gazebo/xmlschema/#interface"
        xmlns:xacro="http://www.ros.org/wiki/xacro">
-  <xacro:macro name="youbot_base_gazebo">
+  <xacro:macro name="youbot_base_gazebo" params="namespace">
     <gazebo reference="youbot_base">
     </gazebo>
@@ -11,8 +11,4 @@
       <kp>1000000</kp>
       <kd>100</kd>
-      <maxContacts>1</maxContacts>
-      <minDepth>0.003</minDepth>
-    </gazebo>
-    <gazebo reference="caster_link_fl">
     </gazebo>
     <!-- front right wheel -->
@@ -20,8 +16,4 @@
       <kp>1000000</kp>
       <kd>100</kd>
-      <maxContacts>1</maxContacts>
-      <minDepth>0.003</minDepth>
-    </gazebo>
-    <gazebo reference="caster_link_fr">
     </gazebo>
     <!-- back left wheel -->
@@ -29,8 +21,4 @@
       <kp>1000000</kp>
       <kd>100</kd>
-      <maxContacts>1</maxContacts>
-      <minDepth>0.003</minDepth>
-    </gazebo>
-    <gazebo reference="caster_link_bl">
     </gazebo>
     <!-- back right wheel -->
@@ -38,8 +26,13 @@
       <kp>1000000</kp>
       <kd>100</kd>
-      <maxContacts>1</maxContacts>
-      <minDepth>0.003</minDepth>
     </gazebo>
-    <gazebo reference="caster_link_br">
+    <gazebo>
+      <plugin name="base_controller" filename="libbase_controller.so">
+        <commandTopic>/cmd_vel</commandTopic>
+        <odometryTopic>odom</odometryTopic>
+        <odometryFrame>odom</odometryFrame>
+        <odometryRate>30.0</odometryRate>
+        <robotBaseFrame>base_footprint</robotBaseFrame>
+      </plugin>
     </gazebo>
   </xacro:macro>

File: urdf/youbot_base/base.transmission.xacro (robot description, xacro)
@@ -7,88 +7,46 @@
   <xacro:property name="caster_mechanical_reduction" value="${624/35 * 80/18}" />
   <xacro:macro name="youbot_base_transmission">
-  <!-- front left wheel -->
-    <transmission name="wheel_trans_fl">
-      <type>transmission_interface/SimpleTransmission</type>
-      <actuator name="wheel_motor_fl">
-        <hardwareInterface>hardware_interface/VelocityJointInterface</hardwareInterface>
-        <mechanicalReduction>${wheel_mechanical_reduction}</mechanicalReduction>
-      </actuator>
-      <joint name="wheel_joint_fl">
-        <hardwareInterface>hardware_interface/VelocityJointInterface</hardwareInterface>
-      </joint>
+    <!--
+    <transmission name="wheel_trans_fl" type="pr2_mechanism_model/SimpleTransmission">
+      <actuator name="wheel_motor_fl"/>
+      <joint name="wheel_joint_fl"/>
+      <mechanicalReduction>79.2380952381</mechanicalReduction>
     </transmission>
-    <transmission name="caster_trans_fl">
-      <type>transmission_interface/SimpleTransmission</type>
-       <actuator name="caster_motor_fl">
-        <hardwareInterface>hardware_interface/VelocityJointInterface</hardwareInterface>
-        <mechanicalReduction>${caster_mechanical_reduction}</mechanicalReduction>
-      </actuator>
-      <joint name="caster_joint_fl">
-        <hardwareInterface>hardware_interface/VelocityJointInterface</hardwareInterface>
-      </joint>
+    <transmission name="caster_trans_fl" type="pr2_mechanism_model/SimpleTransmission">
+      <actuator name="caster_motor_fl"/>
+      <joint name="caster_joint_fl"/>
+      <mechanicalReduction>79.2380952381</mechanicalReduction>
     </transmission>
-    <!-- front right wheel -->
-    <transmission name="wheel_trans_fr">
-      <type>transmission_interface/SimpleTransmission</type>
-      <actuator name="wheel_motor_fr">
-        <hardwareInterface>hardware_interface/VelocityJointInterface</hardwareInterface>
-        <mechanicalReduction>${wheel_mechanical_reduction}</mechanicalReduction>
-      </actuator>
-      <joint name="wheel_joint_fr">
-        <hardwareInterface>hardware_interface/VelocityJointInterface</hardwareInterface>
-      </joint>
+    <transmission name="wheel_trans_fr" type="pr2_mechanism_model/SimpleTransmission">
+      <actuator name="wheel_motor_fr"/>
+      <joint name="wheel_joint_fr"/>
+      <mechanicalReduction>79.2380952381</mechanicalReduction>
     </transmission>
-    <transmission name="caster_trans_fr">
-      <type>transmission_interface/SimpleTransmission</type>
-      <actuator name="caster_motor_fr" >
-        <hardwareInterface>hardware_interface/VelocityJointInterface</hardwareInterface>
-        <mechanicalReduction>${caster_mechanical_reduction}</mechanicalReduction>
-      </actuator>
-      <joint name="caster_joint_fr">
-        <hardwareInterface>hardware_interface/VelocityJointInterface</hardwareInterface>
-      </joint>
+    <transmission name="caster_trans_fr" type="pr2_mechanism_model/SimpleTransmission">
+      <actuator name="caster_motor_fr"/>
+      <joint name="caster_joint_fr"/>
+      <mechanicalReduction>79.2380952381</mechanicalReduction>
     </transmission>
-    <!-- back left wheel -->
-    <transmission name="wheel_trans_bl">
-      <type>transmission_interface/SimpleTransmission</type>
-      <actuator name="wheel_motor_bl" >
-        <hardwareInterface>hardware_interface/VelocityJointInterface</hardwareInterface>
-        <mechanicalReduction>${wheel_mechanical_reduction}</mechanicalReduction>
-      </actuator>
-      <joint name="wheel_joint_bl">
-        <hardwareInterface>hardware_interface/VelocityJointInterface</hardwareInterface>
-      </joint>
+    <transmission name="wheel_trans_bl" type="pr2_mechanism_model/SimpleTransmission">
+      <actuator name="wheel_motor_bl"/>
+      <joint name="wheel_joint_bl"/>
+      <mechanicalReduction>79.2380952381</mechanicalReduction>
     </transmission>
-    <transmission name="caster_trans_bl">
-      <type>transmission_interface/SimpleTransmission</type>
-      <actuator name="caster_motor_bl" >
-        <hardwareInterface>hardware_interface/VelocityJointInterface</hardwareInterface>
-        <mechanicalReduction>${caster_mechanical_reduction}</mechanicalReduction>
-      </actuator>
-      <joint name="caster_joint_bl">
-        <hardwareInterface>hardware_interface/VelocityJointInterface</hardwareInterface>
-      </joint>
+    <transmission name="caster_trans_bl" type="pr2_mechanism_model/SimpleTransmission">
+      <actuator name="caster_motor_bl"/>
+      <joint name="caster_joint_bl"/>
+      <mechanicalReduction>79.2380952381</mechanicalReduction>
     </transmission>
-    <!-- back right wheel -->
-    <transmission name="wheel_trans_br">
-      <type>transmission_interface/SimpleTransmission</type>
-      <actuator name="wheel_motor_br" >
-        <hardwareInterface>hardware_interface/VelocityJointInterface</hardwareInterface>
-        <mechanicalReduction>${wheel_mechanical_reduction}</mechanicalReduction>
-      </actuator>
-      <joint name="wheel_joint_br">
-        <hardwareInterface>hardware_interface/VelocityJointInterface</hardwareInterface>
-      </joint>
+    <transmission name="wheel_trans_br" type="pr2_mechanism_model/SimpleTransmission">
+      <actuator name="wheel_motor_br"/>
+      <joint name="wheel_joint_br"/>
+      <mechanicalReduction>79.2380952381</mechanicalReduction>
     </transmission>
-    <transmission name="caster_trans_br">
-      <type>transmission_interface/SimpleTransmission</type>
-      <actuator name="caster_motor_br" >
-        <hardwareInterface>hardware_interface/VelocityJointInterface</hardwareInterface>
-        <mechanicalReduction>${caster_mechanical_reduction}</mechanicalReduction>
-      </actuator>
-      <joint name="caster_joint_br">
-        <hardwareInterface>hardware_interface/VelocityJointInterface</hardwareInterface>
-      </joint>
+    <transmission name="caster_trans_br" type="pr2_mechanism_model/SimpleTransmission">
+      <actuator name="caster_motor_br"/>
+      <joint name="caster_joint_br"/>
+      <mechanicalReduction>79.2380952381</mechanicalReduction>
     </transmission>
+    -->
   </xacro:macro>
 </robot>
