Commit message: Removed casters and added real youbot wheels. New movement plugin.

File: urdf/youbot_base/base.urdf.xacro (robot description, xacro)
@@ -11,21 +11,12 @@
   <xacro:property name="base_size_z" value="0.100"/>
   <xacro:property name="base_mass" value="22.0"/>
-  <xacro:property name="caster_offset_x" value="0.228"/>
-  <xacro:property name="caster_offset_y" value="0.158"/>
-  <xacro:property name="caster_offset_z" value="-0.034"/>
-  <xacro:property name="caster_mass" value="0.1"/>
-  <xacro:property name="wheel_offset_x" value="0.0"/>
-  <xacro:property name="wheel_offset_y" value="0.0"/>
-  <xacro:property name="wheel_offset_z" value="0.0"/>
+  <property name="wheel_offset_x" value="0.228"  />
+  <property name="wheel_offset_y" value="0.158"  />
+  <property name="wheel_offset_z" value="-0.034" />
   <xacro:property name="wheel_mass" value="1.4"/>
-  <xacro:property name="wheel_radius" value="0.0475"/>
-  <xacro:property name="wheel_length" value="0.005"/>
-  <xacro:property name="caster_joint_damping" value="1.0"/>
-  <xacro:property name="caster_joint_friction" value="1.0"/>
-  <xacro:property name="caster_joint_effort" value="30"/>
-  <xacro:property name="caster_joint_velocity" value="10"/>
-  <xacro:property name="caster_joint_safety_k_velocity" value="10.0"/>
-  <xacro:property name="wheel_joint_damping" value="1.0"/>
-  <xacro:property name="wheel_joint_friction" value="1.0"/>
+  <xacro:property name="wheel_radius" value="0.05"/>
+  <xacro:property name="wheel_length" value="0.07"/>
+  <xacro:property name="wheel_joint_damping" value="0.0"/>
+  <xacro:property name="wheel_joint_friction" value="0.0"/>
   <xacro:property name="wheel_joint_effort" value="30"/>
   <xacro:property name="wheel_joint_velocity" value="10"/>
@@ -74,194 +65,125 @@
     </link>
     <!-- front left wheel -->
-    <joint name="caster_joint_fl" type="continuous">
-      <origin xyz="${caster_offset_x} ${caster_offset_y} ${caster_offset_z}" rpy="0 0 0"/>
-      <axis xyz="0 0 1"/>
-      <limit effort="${caster_joint_effort}" velocity="${caster_joint_velocity}"/>
-      <dynamics damping="${caster_joint_damping}" friction="${caster_joint_friction}"/>
-      <safety_controller k_velocity="${caster_joint_safety_k_velocity}"/>
+    <joint name="wheel_joint_fl" type="continuous">
+      <origin xyz="${wheel_offset_x} ${wheel_offset_y} ${wheel_offset_z}" rpy="0 0 0" />
+      <axis xyz="0 1 0" />
+      <limit effort="${wheel_joint_effort}" velocity="${wheel_joint_velocity}"/>
+      <dynamics damping="${wheel_joint_damping}" friction="${wheel_joint_friction}" />
+      <safety_controller k_velocity="${wheel_joint_safety_k_velocity}" />
       <parent link="${name}_link"/>
-      <child link="caster_link_fl"/>
-    </joint>
-    <link name="caster_link_fl">
-      <inertial>
-        <mass value="${caster_mass}"/>
-        <origin xyz="0 0 0"/>
-        <inertia ixx="0.012411765597" ixy="-0.000711733678" ixz="0.00050272983" iyy="0.015218160428" iyz="-0.000004273467" izz="0.011763977943"/>
-      </inertial>
-    </link>
-    <joint name="wheel_joint_fl" type="continuous">
-      <axis xyz="0 1 0"/>
-      <limit effort="${wheel_joint_effort}" velocity="${wheel_joint_velocity}"/>
-      <origin xyz="${wheel_offset_x} ${wheel_offset_y} ${wheel_offset_z}" rpy="0 0 0"/>
-      <parent link="caster_link_fl"/>
-      <dynamics damping="${wheel_joint_damping}" friction="${wheel_joint_friction}"/>
-      <safety_controller k_velocity="${wheel_joint_safety_k_velocity}"/>
-      <child link="wheel_link_fl"/>
+      <child link="wheel_link_fl" />
     </joint>
     <link name="wheel_link_fl">
       <inertial>
-        <mass value="${wheel_mass}"/>
-        <origin xyz="0 0 0"/>
-        <inertia ixx="0.012411765597" ixy="-0.000711733678" ixz="0.00050272983" iyy="0.015218160428" iyz="-0.000004273467" izz="0.011763977943"/>
+        <mass value="${wheel_mass}" />
+        <origin xyz="0 0 0" />
+        <inertia  ixx="0.012411765597" ixy="-0.000711733678" ixz="0.00050272983"
+                  iyy="0.015218160428" iyz="-0.000004273467" izz="0.011763977943" />
       </inertial>
       <visual>
-        <origin xyz="0 0 0" rpy="0 0 0"/>
-        <!--<mesh filename="package://youbot_description/meshes/youbot_base/youbot_wheel.stl" />-->
+        <origin xyz="0 0 0" rpy="0 0 0" />
         <geometry>
-          <sphere radius="${wheel_radius}"/>
+          <mesh filename="package://youbot_description/meshes/youbot_base/wheel1.dae" />
         </geometry>
-        <material name="youBot/Orange"/>
       </visual>
       <collision>
-        <origin xyz="0 0 0" rpy="${M_PI/2} 0 0"/>
+        <origin xyz="0 0 0" rpy="${M_PI/2} 0 0" />
         <geometry>
-          <cylinder radius="${wheel_radius}" length="${wheel_radius}"/>
+          <cylinder radius="${wheel_radius}" length="${wheel_length}"/>
         </geometry>
       </collision>
     </link>
     <!-- front right wheel -->
-    <joint name="caster_joint_fr" type="continuous">
-      <origin xyz="${caster_offset_x} ${-caster_offset_y} ${caster_offset_z}" rpy="0 0 0"/>
-      <axis xyz="0 0 1"/>
-      <limit effort="${caster_joint_effort}" velocity="${caster_joint_velocity}"/>
-      <dynamics damping="${caster_joint_damping}" friction="${caster_joint_friction}"/>
-      <safety_controller k_velocity="${caster_joint_safety_k_velocity}"/>
+    <joint name="wheel_joint_fr" type="continuous">
+      <origin xyz="${wheel_offset_x} ${-wheel_offset_y} ${wheel_offset_z}" rpy="0 0 0" />
+      <axis xyz="0 1 0" />
+      <limit effort="${wheel_joint_effort}" velocity="${wheel_joint_velocity}"/>
+      <dynamics damping="${wheel_joint_damping}" friction="${wheel_joint_friction}" />
+      <safety_controller k_velocity="${wheel_joint_safety_k_velocity}" />
       <parent link="${name}_link"/>
-      <child link="caster_link_fr"/>
-    </joint>
-    <link name="caster_link_fr">
-      <inertial>
-        <mass value="${caster_mass}"/>
-        <origin xyz="0 0 0"/>
-        <inertia ixx="0.012411765597" ixy="-0.000711733678" ixz="0.00050272983" iyy="0.015218160428" iyz="-0.000004273467" izz="0.011763977943"/>
-      </inertial>
-    </link>
-    <joint name="wheel_joint_fr" type="continuous">
-      <axis xyz="0 1 0"/>
-      <limit effort="${wheel_joint_effort}" velocity="${wheel_joint_velocity}"/>
-      <dynamics damping="${wheel_joint_damping}" friction="${wheel_joint_friction}"/>
-      <safety_controller k_velocity="${wheel_joint_safety_k_velocity}"/>
-      <origin xyz="${wheel_offset_x} ${wheel_offset_y} ${wheel_offset_z}" rpy="0 0 0"/>
-      <parent link="caster_link_fr"/>
-      <child link="wheel_link_fr"/>
+      <child link="wheel_link_fr" />
     </joint>
     <link name="wheel_link_fr">
       <inertial>
-        <mass value="${wheel_mass}"/>
-        <origin xyz="0 0 0"/>
-        <inertia ixx="0.012411765597" ixy="-0.000711733678" ixz="0.00050272983" iyy="0.015218160428" iyz="-0.000004273467" izz="0.011763977943"/>
+        <mass value="${wheel_mass}" />
+        <origin xyz="0 0 0" />
+        <inertia  ixx="0.012411765597" ixy="-0.000711733678" ixz="0.00050272983"
+                  iyy="0.015218160428" iyz="-0.000004273467" izz="0.011763977943" />
       </inertial>
       <visual>
-        <origin xyz="0 0 0" rpy="0 0 0"/>
+        <origin xyz="0 0 0" rpy="0 0 0" />
         <geometry>
-          <!--<mesh filename="package://youbot_description/meshes/youbot_base/youbot_wheel.stl" />-->
-          <sphere radius="${wheel_radius}"/>
+          <mesh filename="package://youbot_description/meshes/youbot_base/wheel2.dae" />
         </geometry>
-        <material name="youBot/Orange"/>
       </visual>
       <collision>
-        <origin xyz="0 0 0" rpy="${M_PI/2} 0 0"/>
+        <origin xyz="0 0 0" rpy="${M_PI/2} 0 0" />
         <geometry>
-          <cylinder radius="${wheel_radius}" length="${wheel_radius}"/>
+          <cylinder radius="${wheel_radius}" length="${wheel_length}"/>
         </geometry>
       </collision>
     </link>
     <!-- back left wheel -->
-    <joint name="caster_joint_bl" type="continuous">
-      <origin xyz="${-caster_offset_x} ${caster_offset_y} ${caster_offset_z}" rpy="0 0 0"/>
-      <axis xyz="0 0 1"/>
-      <limit effort="${caster_joint_effort}" velocity="${caster_joint_velocity}"/>
-      <dynamics damping="${caster_joint_damping}" friction="${caster_joint_friction}"/>
-      <safety_controller k_velocity="${caster_joint_safety_k_velocity}"/>
+    <joint name="wheel_joint_bl" type="continuous">
+      <origin xyz="${-wheel_offset_x} ${wheel_offset_y} ${wheel_offset_z}" rpy="0 0 0" />
+      <axis xyz="0 1 0" />
+      <limit effort="${wheel_joint_effort}" velocity="${wheel_joint_velocity}"/>
+      <dynamics damping="${wheel_joint_damping}" friction="${wheel_joint_friction}" />
+      <safety_controller k_velocity="${wheel_joint_safety_k_velocity}" />
       <parent link="${name}_link"/>
-      <child link="caster_link_bl"/>
-    </joint>
-    <link name="caster_link_bl">
-      <inertial>
-        <mass value="${caster_mass}"/>
-        <origin xyz="0 0 0"/>
-        <inertia ixx="0.012411765597" ixy="-0.000711733678" ixz="0.00050272983" iyy="0.015218160428" iyz="-0.000004273467" izz="0.011763977943"/>
-      </inertial>
-    </link>
-    <joint name="wheel_joint_bl" type="continuous">
-      <axis xyz="0 1 0"/>
-      <limit effort="10" velocity="10"/>
-      <limit effort="${wheel_joint_effort}" velocity="${wheel_joint_velocity}"/>
-      <dynamics damping="${wheel_joint_damping}" friction="${wheel_joint_friction}"/>
-      <safety_controller k_velocity="${wheel_joint_safety_k_velocity}"/>
-      <origin xyz="${wheel_offset_x} ${wheel_offset_y} ${wheel_offset_z}" rpy="0 0 0"/>
-      <parent link="caster_link_bl"/>
-      <child link="wheel_link_bl"/>
+      <child link="wheel_link_bl" />
     </joint>
     <link name="wheel_link_bl">
       <inertial>
-        <mass value="${wheel_mass}"/>
-        <origin xyz="0 0 0"/>
-        <inertia ixx="0.012411765597" ixy="-0.000711733678" ixz="0.00050272983" iyy="0.015218160428" iyz="-0.000004273467" izz="0.011763977943"/>
+        <mass value="${wheel_mass}" />
+        <origin xyz="0 0 0" />
+        <inertia  ixx="0.012411765597" ixy="-0.000711733678" ixz="0.00050272983"
+                  iyy="0.015218160428" iyz="-0.000004273467" izz="0.011763977943" />
       </inertial>
       <visual>
-        <origin xyz="0 0 0" rpy="0 0 0"/>
+        <origin xyz="0 0 0" rpy="0 0 0" />
         <geometry>
-          <!--<mesh filename="package://youbot_description/meshes/youbot_base/youbot_wheel.stl" />-->
-          <sphere radius="${wheel_radius}"/>
+          <mesh filename="package://youbot_description/meshes/youbot_base/wheel2.dae" />
         </geometry>
-        <material name="youBot/Orange"/>
       </visual>
       <collision>
-        <origin xyz="0 0 0" rpy="${M_PI/2} 0 0"/>
+        <origin xyz="0 0 0" rpy="${M_PI/2} 0 0" />
         <geometry>
-          <cylinder radius="${wheel_radius}" length="${wheel_radius}"/>
+          <cylinder radius="${wheel_radius}" length="${wheel_length}"/>
         </geometry>
       </collision>
     </link>
     <!-- back right wheel -->
-    <joint name="caster_joint_br" type="continuous">
-      <origin xyz="${-caster_offset_x} ${-caster_offset_y} ${caster_offset_z}" rpy="0 0 0"/>
-      <axis xyz="0 0 1"/>
-      <limit effort="${caster_joint_effort}" velocity="${caster_joint_velocity}"/>
-      <dynamics damping="${caster_joint_damping}" friction="${caster_joint_friction}"/>
-      <safety_controller k_velocity="${caster_joint_safety_k_velocity}"/>
+    <joint name="wheel_joint_br" type="continuous">
+      <origin xyz="${-wheel_offset_x} ${-wheel_offset_y} ${wheel_offset_z}" rpy="0 0 0" />
+      <axis xyz="0 1 0" />
+      <limit effort="${wheel_joint_effort}" velocity="${wheel_joint_velocity}"/>
+      <dynamics damping="${wheel_joint_damping}" friction="${wheel_joint_friction}" />
+      <safety_controller k_velocity="${wheel_joint_safety_k_velocity}" />
       <parent link="${name}_link"/>
-      <child link="caster_link_br"/>
-    </joint>
-    <link name="caster_link_br">
-      <inertial>
-        <mass value="${caster_mass}"/>
-        <origin xyz="0 0 0"/>
-        <inertia ixx="0.012411765597" ixy="-0.000711733678" ixz="0.00050272983" iyy="0.015218160428" iyz="-0.000004273467" izz="0.011763977943"/>
-      </inertial>
-    </link>
-    <joint name="wheel_joint_br" type="continuous">
-      <axis xyz="0 1 0"/>
-      <limit effort="${wheel_joint_effort}" velocity="${wheel_joint_velocity}"/>
-      <dynamics damping="${wheel_joint_damping}" friction="${wheel_joint_friction}"/>
-      <safety_controller k_velocity="${wheel_joint_safety_k_velocity}"/>
-      <origin xyz="${wheel_offset_x} ${wheel_offset_y} ${wheel_offset_z}" rpy="0 0 0"/>
-      <parent link="caster_link_br"/>
-      <child link="wheel_link_br"/>
+      <child link="wheel_link_br" />
     </joint>
     <link name="wheel_link_br">
       <inertial>
-        <mass value="${wheel_mass}"/>
-        <origin xyz="0 0 0"/>
-        <inertia ixx="0.012411765597" ixy="-0.000711733678" ixz="0.00050272983" iyy="0.015218160428" iyz="-0.000004273467" izz="0.011763977943"/>
+        <mass value="${wheel_mass}" />
+        <origin xyz="0 0 0" />
+        <inertia  ixx="0.012411765597" ixy="-0.000711733678" ixz="0.00050272983"
+                  iyy="0.015218160428" iyz="-0.000004273467" izz="0.011763977943" />
       </inertial>
       <visual>
-        <origin xyz="0 0 0" rpy="0 0 0"/>
+        <origin xyz="0 0 0" rpy="0 0 0" />
         <geometry>
-          <!--<mesh filename="package://youbot_description/meshes/youbot_base/youbot_wheel.stl" />-->
-          <sphere radius="${wheel_radius}"/>
+          <mesh filename="package://youbot_description/meshes/youbot_base/wheel1.dae" />
         </geometry>
-        <material name="youBot/Orange"/>
       </visual>
       <collision>
-        <origin xyz="0 0 0" rpy="${M_PI/2} 0 0"/>
+        <origin xyz="0 0 0" rpy="${M_PI/2} 0 0" />
         <geometry>
-          <cylinder radius="${wheel_radius}" length="${wheel_radius}"/>
+          <cylinder radius="${wheel_radius}" length="${wheel_length}"/>
         </geometry>
       </collision>
     </link>
     <!-- extensions -->
-    <xacro:youbot_base_gazebo/>
+    <xacro:youbot_base_gazebo namespace="gazebo"/>
     <xacro:youbot_base_transmission/>
   </xacro:macro>

File: urdf/youbot_gripper/grasp_fix_plugin.urdf.xacro (robot description, xacro)
@@ -21,5 +21,5 @@
                 <grip_count_threshold>4</grip_count_threshold>
                 <max_grip_count>8</max_grip_count>
-                <release_tolerance>0.0005</release_tolerance>
+                <release_tolerance>0.01</release_tolerance>
                 <disable_collisions_on_attach>false</disable_collisions_on_attach>
                 <contact_topic>__default_topic__</contact_topic>

File: urdf/youbot_gripper/gripper.gazebo.xacro (robot description, xacro)
@@ -14,4 +14,9 @@
 			<turnGravityOff>false</turnGravityOff>
 			<selfCollide>true</selfCollide>
+			<!--
+			<mu1>100.0</mu1>
+			<mu2>100.0</mu2>
+			<minDepth>0.003</minDepth>
+			-->
 		</gazebo>
 		<gazebo reference="${name}_finger_r_link">
@@ -19,4 +24,9 @@
 			<turnGravityOff>false</turnGravityOff>
 			<selfCollide>true</selfCollide>
+			<!--
+			<mu1>100.0</mu1>
+			<mu2>100.0</mu2>
+			<minDepth>0.003</minDepth>
+			-->
 		</gazebo>
 	</xacro:macro>
