Commit message: Changes to use realsense_gazebo_plugin

File: urdf/sensors/intel_d435.gazebo.xacro (robot description, xacro)
@@ -4,53 +4,91 @@
       xmlns:interface="http://playerstage.sourceforge.net/gazebo/xmlschema/#interface"
       xmlns:xacro="http://www.ros.org/wiki/xacro">
-  <xacro:macro name="intel_d435_gazebo" params="name">
-    <gazebo reference="${name}_camera">
-      <material>Gazebo/Grey</material>
-      <sensor type="depth" name="${name}_depth_frame_sensor">
-        <always_on>true</always_on>
-        <update_rate>30.0</update_rate>
-        <camera>
-          <horizontal_fov>${87.0*M_PI/180.0}</horizontal_fov>
+  <xacro:macro name="gazebo_d435" params="camera_name reference_link topics_ns depth_optical_frame color_optical_frame infrared1_optical_frame infrared2_optical_frame" >
+    <!-- Load parameters to model's main link-->
+    <xacro:property name="deg_to_rad" value="0.01745329251994329577" />
+    <gazebo reference="${reference_link}">
+      <self_collide>0</self_collide>
+      <enable_wind>0</enable_wind>
+      <kinematic>0</kinematic>
+      <gravity>1</gravity>
+      <!--<mu>1</mu>-->
+      <mu2>1</mu2>
+      <fdir1>0 0 0</fdir1>
+      <!--<slip1>0</slip1>
+      <slip2>0</slip2>-->
+      <kp>1e+13</kp>
+      <kd>1</kd>
+      <!--<max_vel>0.01</max_vel>
+      <min_depth>0</min_depth>-->
+      <sensor name="${camera_name}color" type="camera">
+        <camera name="${camera_name}">
+          <horizontal_fov>${69.4*deg_to_rad}</horizontal_fov>
           <image>
-            <format>R8G8B8</format>
+            <width>1920</width>
+            <height>1080</height>
+            <format>RGB_INT8</format>
+          </image>
+          <clip>
+            <near>0.1</near>
+            <far>100</far>
+          </clip>
+          <noise>
+            <type>gaussian</type>
+            <mean>0.0</mean>
+            <stddev>0.007</stddev>
+          </noise>
+        </camera>
+        <always_on>1</always_on>
+        <update_rate>30</update_rate>
+        <visualize>1</visualize>
+      </sensor>
+      <sensor name="${camera_name}ired1" type="camera">
+        <camera name="${camera_name}">
+          <horizontal_fov>${85.2*deg_to_rad}</horizontal_fov>
+          <image>
             <width>1280</width>
             <height>720</height>
+            <format>L_INT8</format>
           </image>
           <clip>
-            <near>0.105</near>
-            <far>5</far>
+            <near>0.1</near>
+            <far>100</far>
           </clip>
+          <noise>
+            <type>gaussian</type>
+            <mean>0.0</mean>
+            <stddev>0.05</stddev>
+          </noise>
         </camera>
-        <plugin name="${name}_depth_frame_controller" filename="libgazebo_ros_openni_kinect.so">
-          <baseline>0.2</baseline>
-          <alwaysOn>true</alwaysOn>
-          <updateRate>30.0</updateRate>
-          <cameraName>${name}_depth</cameraName>
-          <imageTopicName>/${name}/ir/image_raw</imageTopicName>
-          <cameraInfoTopicName>/${name}/ir/camera_info</cameraInfoTopicName>
-          <depthImageTopicName>/${name}/depth/image_raw</depthImageTopicName>
-          <depthImageCameraInfoTopicName>/${name}/depth/camera_info</depthImageCameraInfoTopicName>
-          <pointCloudTopicName>/${name}/depth/points</pointCloudTopicName>
-          <frameName>${name}_depth_optical_frame</frameName>
-          <pointCloudCutoff>0.105</pointCloudCutoff>
-          <distortionK1>0.00000001</distortionK1>
-          <distortionK2>0.00000001</distortionK2>
-          <distortionK3>0.00000001</distortionK3>
-          <distortionT1>0.00000001</distortionT1>
-          <distortionT2>0.00000001</distortionT2>
-          <CxPrime>0</CxPrime>
-          <Cx>0</Cx>
-          <Cy>0</Cy>
-          <focalLength>0</focalLength>
-          <hackBaseline>0</hackBaseline>
-        </plugin>
+        <always_on>1</always_on>
+        <update_rate>90</update_rate>
+        <visualize>0</visualize>
       </sensor>
-      <sensor type="depth" name="${name}_rgb_frame_sensor">
-        <always_on>true</always_on>
-        <update_rate>30.0</update_rate>
-        <camera>
-          <horizontal_fov>${87.0*M_PI/180.0}</horizontal_fov>
+      <sensor name="${camera_name}ired2" type="camera">
+        <camera name="${camera_name}">
+          <horizontal_fov>${85.2*deg_to_rad}</horizontal_fov>
           <image>
-            <format>R8G8B8</format>
+            <width>1280</width>
+            <height>720</height>
+            <format>L_INT8</format>
+          </image>
+          <clip>
+            <near>0.1</near>
+            <far>100</far>
+          </clip>
+          <noise>
+            <type>gaussian</type>
+            <mean>0.0</mean>
+            <stddev>0.05</stddev>
+          </noise>
+        </camera>
+        <always_on>1</always_on>
+        <update_rate>90</update_rate>
+        <visualize>0</visualize>
+      </sensor>
+      <sensor name="${camera_name}depth" type="depth">
+        <camera name="${camera_name}">
+          <horizontal_fov>${85.2*deg_to_rad}</horizontal_fov>
+          <image>
             <width>1280</width>
             <height>720</height>
@@ -58,31 +96,41 @@
           <clip>
             <near>0.1</near>
-            <far>5</far>
+            <far>100</far>
           </clip>
+          <noise>
+            <type>gaussian</type>
+            <mean>0.0</mean>
+            <stddev>0.100</stddev>
+          </noise>
         </camera>
-        <plugin name="${name}_rgb_frame_controller" filename="libgazebo_ros_openni_kinect.so">
-          <baseline>0.2</baseline>
-          <alwaysOn>true</alwaysOn>
-          <updateRate>30.0</updateRate>
-          <cameraName>${name}_rgb</cameraName>
-          <imageTopicName>/${name}/rgb/image_raw</imageTopicName>
-          <cameraInfoTopicName>/${name}/rgb/camera_info</cameraInfoTopicName>
-          <depthImageTopicName>/${name}/depth_registered/image_raw</depthImageTopicName>
-          <depthImageCameraInfoTopicName>/${name}/depth_registered/camera_info</depthImageCameraInfoTopicName>
-          <pointCloudTopicName>/${name}/depth_registered/points</pointCloudTopicName>
-          <frameName>${name}_rgb_optical_frame</frameName>
-          <pointCloudCutoff>0.1</pointCloudCutoff>
-          <distortionK1>0.00000001</distortionK1>
-          <distortionK2>0.00000001</distortionK2>
-          <distortionK3>0.00000001</distortionK3>
-          <distortionT1>0.00000001</distortionT1>
-          <distortionT2>0.00000001</distortionT2>
-          <CxPrime>0</CxPrime>
-          <Cx>0</Cx>
-          <Cy>0</Cy>
-          <focalLength>0</focalLength>
-          <hackBaseline>0</hackBaseline>
-        </plugin>
+        <always_on>1</always_on>
+        <update_rate>90</update_rate>
+        <visualize>0</visualize>
       </sensor>
+    </gazebo>
+    <gazebo>
+      <plugin name="${topics_ns}" filename="librealsense_gazebo_plugin.so">
+        <prefix>${camera_name}</prefix>
+        <depthUpdateRate>30.0</depthUpdateRate>
+        <colorUpdateRate>30.0</colorUpdateRate>
+        <infraredUpdateRate>30.0</infraredUpdateRate>
+        <depthTopicName>depth/image_raw</depthTopicName>
+        <depthCameraInfoTopicName>depth/camera_info</depthCameraInfoTopicName>
+        <colorTopicName>color/image_raw</colorTopicName>
+        <colorCameraInfoTopicName>color/camera_info</colorCameraInfoTopicName>
+        <infrared1TopicName>infra1/image_raw</infrared1TopicName>
+        <infrared1CameraInfoTopicName>infra1/camera_info</infrared1CameraInfoTopicName>
+        <infrared2TopicName>infra2/image_raw</infrared2TopicName>
+        <infrared2CameraInfoTopicName>infra2/camera_info</infrared2CameraInfoTopicName>
+        <colorOpticalframeName>${color_optical_frame}</colorOpticalframeName>
+        <depthOpticalframeName>${depth_optical_frame}</depthOpticalframeName>
+        <infrared1OpticalframeName>${infrared1_optical_frame}</infrared1OpticalframeName>
+        <infrared2OpticalframeName>${infrared2_optical_frame}</infrared2OpticalframeName>
+        <rangeMinDepth>0.2</rangeMinDepth>
+        <rangeMaxDepth>10.0</rangeMaxDepth>
+        <pointCloud>true</pointCloud>
+        <pointCloudTopicName>depth/points</pointCloudTopicName>
+        <pointCloudCutoff>0.2</pointCloudCutoff>
+      </plugin>
     </gazebo>
   </xacro:macro>
