Commit message: Changes to use realsense_gazebo_plugin

File: urdf/sensors/intel_d435.urdf.xacro (robot description, xacro)
@@ -7,163 +7,150 @@
 -->
 <root xmlns:xacro="http://playerstage.sourceforge.net/gazebo/xmlschema/#interface">
-  <xacro:include filename="$(find youbot_description)/urdf/sensors/intel_d435.gazebo.xacro" />
-  <xacro:property name="M_PI" value="3.1415926535897931" />
-  <!-- The following values are approximate, and the camera node
-   publishing TF values with actual calibrated camera extrinsic values -->
-  <xacro:property name="d435_cam_depth_to_left_ir_offset" value="-0.025"/>
-  <xacro:property name="d435_cam_depth_to_right_ir_offset" value="0.025"/>
-  <xacro:property name="d435_cam_depth_to_fisheye_offset" value="0.040"/>
-  <!-- The following values model the aluminum peripherial case for the
-    D435 camera, with the camera joint represented by the actual
-    peripherial camera tripod mount -->
-  <xacro:property name="d435_cam_width" value="0.090"/>
-  <xacro:property name="d435_cam_height" value="0.025"/>
-  <xacro:property name="d435_cam_depth" value="0.02505"/>
-  <xacro:property name="d435_cam_mount_from_center_offset" value="0.0149"/>
-  <!-- The following offset is relative the the physical D435 camera peripherial
-    camera tripod mount -->
-  <xacro:property name="d435_cam_depth_px" value="${d435_cam_mount_from_center_offset}"/>
-  <xacro:property name="d435_cam_depth_py" value="-0.0075"/>
-  <xacro:property name="d435_cam_depth_pz" value="${d435_cam_height/2}"/>
-  <material name="aluminum">
-    <color rgba="0.5 0.5 0.5 1"/>
-  </material>
-  <xacro:macro name="intel_d435" params="name parent *origin tilt">
-    <link name="${name}_foot_link">
-      <inertial>
-        <mass value="0.05" />
-        <origin xyz="0 0 0" rpy="0 0 0"/>
-        <inertia ixx="0.0001" ixy="0" ixz="0" iyy="0.0001" iyz="0" izz="0.0001" />
-      </inertial>
-      <!--
-      <visual>
-        <origin xyz="0 0 0" rpy="${M_PI/2} 0 ${M_PI/2}" />
-        <geometry>
-          <mesh filename="package://youbot_description/meshes/sensors/d435_mount.dae"/>
-        </geometry>
-        <material name="Black" />
-      </visual>
-      <collision>
-        <origin xyz="0 0 0" rpy="${M_PI/2} 0 ${M_PI/2}" />
-        <geometry>
-          <mesh filename="package://youbot_description/meshes/sensors/d435_mount.dae"/>
-        </geometry>
-      </collision >
-      -->
-    </link>
-    <joint name="${name}_foot_joint" type="fixed">
-      <xacro:insert_block name="origin" />
-      <parent link="${parent}"/>
-      <child link="${name}_foot_link"/>
-    </joint>
-    <link name="${name}_tilt_link">
-      <inertial>
-        <mass value="0.01" />
-        <origin xyz="0 0 0" rpy="0 0 0"/>
-        <inertia ixx="0.0001" ixy="0" ixz="0" iyy="0.0001" iyz="0" izz="0.0001" />
-      </inertial>
-      <visual>
-        <origin xyz="0 0 0.0075" rpy="0 0 0" />
-        <geometry>
-          <cylinder length="0.05" radius="0.003" />
-        </geometry>
-        <material name="aluminum"/>
-      </visual>
-      <collision>
-        <origin xyz="0 0 0.0075" rpy="0 0 0" />
-        <geometry>
-          <cylinder length="0.05" radius="0.003" />
-        </geometry>
-        <material name="aluminum"/>
-      </collision >
-    </link>
-    <joint name="intel_d435_tilt_joint" type="fixed">
-      <parent link="${name}_foot_link"/>
-      <child link="${name}_tilt_link"/>
-      <!--<axis xyz="0 1 0"/>-->
-      <origin xyz="0 0 0.0075" rpy="0 ${tilt} 0"/>
-      <!--<limit effort="100" lower="-0.541052068" upper="0.541052068" velocity="1.0"/>-->
-    </joint>
-    <!-- camera body, with origin at bottom screw mount -->
-    <joint name="${name}_camera_joint" type="fixed">
-      <origin xyz="0 0 0.03" rpy="0 0 0" />
-      <parent link="${name}_tilt_link"/>
-      <child link="${name}_camera" />
-    </joint>
-    <link name="${name}_camera">
-      <visual>
-      <origin xyz="${d435_cam_mount_from_center_offset} 0.0 ${d435_cam_height/2}" rpy="${M_PI/2} 0 ${M_PI/2}"/>
-        <geometry>
-          <!-- <box size="${d435_cam_width} ${d435_cam_height} ${d435_cam_depth}"/> -->
-	  <mesh filename="package://youbot_description/meshes/sensors/d435.dae" />
-        </geometry>
-        <material name="aluminum"/>
-      </visual>
-      <collision>
-        <origin xyz="0.0 0.0 ${d435_cam_height/2}" rpy="0 0 0"/>
-        <geometry>
-        <box size="${d435_cam_depth} ${d435_cam_width} ${d435_cam_height}"/>
-        </geometry>
-      </collision>
-      <inertial>
-        <!-- The following are not reliable values, and should not be used for modeling -->
-        <mass value="0.564" />
-        <origin xyz="0 0 0" />
-        <inertia ixx="0.003881243" ixy="0.0" ixz="0.0" iyy="0.000498940" iyz="0.0" izz="0.003879257" />
-      </inertial>
-    </link>
-    <!-- camera depth joints and links -->
-    <joint name="${name}_depth_joint" type="fixed">
-      <origin xyz="${d435_cam_depth_px} ${d435_cam_depth_py} ${d435_cam_depth_pz}" rpy="0 0 0"/>
-      <parent link="${name}_camera"/>
-      <child link="${name}_depth_frame" />
-    </joint>
-    <link name="${name}_depth_frame"/>
-    <joint name="${name}_depth_optical_joint" type="fixed">
-      <origin xyz="0 0 0" rpy="${-M_PI/2} 0 ${-M_PI/2}" />
-      <parent link="${name}_depth_frame" />
-      <child link="${name}_depth_optical_frame" />
-    </joint>
-    <link name="${name}_depth_optical_frame"/>
-    <!-- camera left IR joints and links -->
-    <joint name="${name}_left_ir_joint" type="fixed">
-      <origin xyz="0 ${d435_cam_depth_to_left_ir_offset} 0" rpy="0 0 0" />
-      <parent link="${name}_depth_frame" />
-      <child link="${name}_left_ir_frame" />
-    </joint>
-    <link name="${name}_left_ir_frame"/>
-    <joint name="${name}_left_ir_optical_joint" type="fixed">
-      <origin xyz="0 0 0" rpy="${-M_PI/2} 0 ${-M_PI/2}" />
-      <parent link="${name}_left_ir_frame" />
-      <child link="${name}_left_ir_optical_frame" />
-    </joint>
-    <link name="${name}_left_ir_optical_frame"/>
-    <!-- camera right IR joints and links -->
-    <joint name="${name}_right_ir_joint" type="fixed">
-      <origin xyz="0 ${d435_cam_depth_to_right_ir_offset} 0" rpy="0 0 0" />
-      <parent link="${name}_depth_frame" />
-      <child link="${name}_right_ir_frame" />
-    </joint>
-    <link name="${name}_right_ir_frame"/>
-    <joint name="${name}_right_ir_optical_joint" type="fixed">
-      <origin xyz="0 0 0" rpy="${-M_PI/2} 0 ${-M_PI/2}" />
-      <parent link="${name}_right_ir_frame" />
-      <child link="${name}_right_ir_optical_frame" />
-    </joint>
-    <link name="${name}_right_ir_optical_frame"/>
-    <!-- camera fisheye joints and links -->
-    <joint name="${name}_fisheye_joint" type="fixed">
-      <origin xyz="0 ${d435_cam_depth_to_fisheye_offset} 0" rpy="0 0 0" />
-      <parent link="${name}_depth_frame" />
-      <child link="${name}_fisheye_frame" />
-    </joint>
-    <link name="${name}_fisheye_frame"/>
-    <joint name="${name}_fisheye_optical_joint" type="fixed">
-      <origin xyz="0 0 0" rpy="${-M_PI/2} 0 ${-M_PI/2}" />
-      <parent link="${name}_fisheye_frame" />
-      <child link="${name}_fisheye_optical_frame" />
-    </joint>
-    <link name="${name}_fisheye_optical_frame"/>
-    <xacro:intel_d435_gazebo name="${name}" />
-  </xacro:macro>
+    <xacro:include filename="$(find youbot_description)/urdf/sensors/intel_d435.gazebo.xacro"/>
+    <xacro:property name="M_PI" value="3.1415926535897931"/>
+    <!-- The following values are approximate, and the camera node
+     publishing TF values with actual calibrated camera extrinsic values -->
+    <xacro:property name="d435_cam_depth_to_left_ir_offset" value="0.0"/>
+    <xacro:property name="d435_cam_depth_to_right_ir_offset" value="-0.050"/>
+    <xacro:property name="d435_cam_depth_to_color_offset" value="0.0"/>
+    <!-- The following values model the aluminum peripherial case for the
+      D435 camera, with the camera joint represented by the actual
+      peripherial camera tripod mount -->
+    <xacro:property name="d435_cam_width" value="0.090"/>
+    <xacro:property name="d435_cam_height" value="0.025"/>
+    <xacro:property name="d435_cam_depth" value="0.02505"/>
+    <xacro:property name="d435_cam_mount_from_center_offset" value="0.0149"/>
+    <!-- The following offset is relative the the physical D435 camera peripherial
+      camera tripod mount -->
+    <xacro:property name="d435_cam_depth_px" value="${d435_cam_mount_from_center_offset}"/>
+    <xacro:property name="d435_cam_depth_py" value="-0.0075"/>
+    <xacro:property name="d435_cam_depth_pz" value="${d435_cam_height/2}"/>
+    <material name="aluminum">
+        <color rgba="0.5 0.5 0.5 1"/>
+    </material>
+    <xacro:macro name="intel_d435" params="name parent topics_ns:=depth_cam *origin tilt">
+        <link name="${name}_foot_link">
+            <inertial>
+                <mass value="0.05"/>
+                <origin xyz="0 0 0" rpy="0 0 0"/>
+                <inertia ixx="0.0001" ixy="0" ixz="0" iyy="0.0001" iyz="0" izz="0.0001"/>
+            </inertial>
+        </link>
+        <joint name="${name}_foot_joint" type="fixed">
+            <xacro:insert_block name="origin"/>
+            <parent link="${parent}"/>
+            <child link="${name}_foot_link"/>
+        </joint>
+        <link name="${name}_tilt_link">
+            <inertial>
+                <mass value="0.01"/>
+                <origin xyz="0 0 0" rpy="0 0 0"/>
+                <inertia ixx="0.0001" ixy="0" ixz="0" iyy="0.0001" iyz="0" izz="0.0001"/>
+            </inertial>
+            <visual>
+                <origin xyz="0 0 0.0075" rpy="0 0 0"/>
+                <geometry>
+                    <cylinder length="0.05" radius="0.003"/>
+                </geometry>
+                <material name="aluminum"/>
+            </visual>
+            <collision>
+                <origin xyz="0 0 0.0075" rpy="0 0 0"/>
+                <geometry>
+                    <cylinder length="0.05" radius="0.003"/>
+                </geometry>
+                <material name="aluminum"/>
+            </collision>
+        </link>
+        <joint name="intel_d435_tilt_joint" type="fixed">
+            <parent link="${name}_foot_link"/>
+            <child link="${name}_tilt_link"/>
+            <!--<axis xyz="0 1 0"/>-->
+            <origin xyz="0 0 0.0075" rpy="0 ${tilt} 0"/>
+            <!--<limit effort="100" lower="-0.541052068" upper="0.541052068" velocity="1.0"/>-->
+        </joint>
+        <!-- camera body, with origin at bottom screw mount -->
+        <joint name="${name}_camera_joint" type="fixed">
+            <origin xyz="0 0 0.03" rpy="0 0 0"/>
+            <parent link="${name}_tilt_link"/>
+            <child link="${name}_camera"/>
+        </joint>
+        <link name="${name}_camera">
+            <visual>
+                <origin xyz="${d435_cam_mount_from_center_offset} 0.0 0" rpy="${M_PI/2} 0 ${M_PI/2}"/>
+                <geometry>
+                    <mesh filename="package://youbot_description/meshes/sensors/d435.dae"/>
+                </geometry>
+            </visual>
+            <collision>
+                <origin xyz="0.0 0.0 ${d435_cam_height/2}" rpy="0 0 0"/>
+                <geometry>
+                    <mesh filename="package://youbot_description/meshes/sensors/d435.dae"/>
+                </geometry>
+            </collision>
+            <inertial>
+                <!-- The following are not reliable values, and should not be used for modeling -->
+                <mass value="0.564"/>
+                <origin xyz="0 0 0"/>
+                <inertia ixx="0.003881243" ixy="0.0" ixz="0.0" iyy="0.000498940" iyz="0.0" izz="0.003879257"/>
+            </inertial>
+        </link>
+        <!-- camera depth joints and links -->
+        <joint name="${name}_depth_joint" type="fixed">
+            <origin xyz="0 0 0" rpy="0 0 0"/>
+            <parent link="${name}_camera"/>
+            <child link="${name}_depth_frame"/>
+        </joint>
+        <link name="${name}_depth_frame"/>
+        <joint name="${name}_depth_optical_joint" type="fixed">
+            <origin xyz="0 0 0" rpy="${-M_PI/2} 0 ${-M_PI/2}"/>
+            <parent link="${name}_depth_frame"/>
+            <child link="${name}_depth_optical_frame"/>
+        </joint>
+        <link name="${name}_depth_optical_frame"/>
+        <!-- camera left IR joints and links -->
+        <joint name="${name}_left_ir_joint" type="fixed">
+            <origin xyz="0 ${d435_cam_depth_to_left_ir_offset} 0" rpy="0 0 0"/>
+            <parent link="${name}_depth_frame"/>
+            <child link="${name}_left_ir_frame"/>
+        </joint>
+        <link name="${name}_left_ir_frame"/>
+        <joint name="${name}_left_ir_optical_joint" type="fixed">
+            <origin xyz="0 0 0" rpy="${-M_PI/2} 0 ${-M_PI/2}"/>
+            <parent link="${name}_left_ir_frame"/>
+            <child link="${name}_left_ir_optical_frame"/>
+        </joint>
+        <link name="${name}_left_ir_optical_frame"/>
+        <!-- camera right IR joints and links -->
+        <joint name="${name}_right_ir_joint" type="fixed">
+            <origin xyz="0 ${d435_cam_depth_to_right_ir_offset} 0" rpy="0 0 0"/>
+            <parent link="${name}_depth_frame"/>
+            <child link="${name}_right_ir_frame"/>
+        </joint>
+        <link name="${name}_right_ir_frame"/>
+        <joint name="${name}_right_ir_optical_joint" type="fixed">
+            <origin xyz="0 0 0" rpy="${-M_PI/2} 0 ${-M_PI/2}"/>
+            <parent link="${name}_right_ir_frame"/>
+            <child link="${name}_right_ir_optical_frame"/>
+        </joint>
+        <link name="${name}_right_ir_optical_frame"/>
+        <!-- camera color joints and links -->
+        <joint name="${name}_color_joint" type="fixed">
+            <origin xyz="0 ${d435_cam_depth_to_color_offset} 0" rpy="0 0 0"/>
+            <parent link="${name}_depth_frame"/>
+            <child link="${name}_color_frame"/>
+        </joint>
+        <link name="${name}_color_frame"/>
+        <joint name="${name}_color_optical_joint" type="fixed">
+            <origin xyz="0 0 0" rpy="${-M_PI/2} 0 ${-M_PI/2}"/>
+            <parent link="${name}_color_frame"/>
+            <child link="${name}_color_optical_frame"/>
+        </joint>
+        <link name="${name}_color_optical_frame"/>
+        <xacro:gazebo_d435 camera_name="${name}" reference_link="${name}_camera" topics_ns="${topics_ns}"
+                           depth_optical_frame="${name}_depth_optical_frame"
+                           color_optical_frame="${name}_color_optical_frame"
+                           infrared1_optical_frame="${name}_left_ir_optical_frame"
+                           infrared2_optical_frame="${name}_right_ir_optical_frame"/>
+    </xacro:macro>
 </root>
