Commit message: Code to fix interia problem.

File: urdf/youbot_base/base.urdf.xacro (robot description, xacro)
@@ -57,4 +57,11 @@
       <parent link="${name}_footprint"/>
     </joint>
+    <!-- Fix inertia warning
+    <link name="dummy"></link>
+    <joint name="dummy_joint" type="fixed">
+      <parent link="dummy"/>
+      <child link="base_footprint"/>
+    </joint>
+    Fix warning -->
     <link name="${name}_link">
       <inertial>
