Commit message: Fixed unneccesary torsional frciction and mu-factors. They led to abrupt stopping when planning.

File: urdf/youbot_base/base.gazebo.xacro (robot description, xacro)
@@ -11,19 +11,6 @@
       <kp>1000000</kp>
       <kd>100</kd>
-      <mu1>100000.0</mu1>
-      <mu2>100000.0</mu2>
       <maxContacts>1</maxContacts>
       <minDepth>0.003</minDepth>
-      <collision name="wheel_link_fl_collision">
-        <surface>
-          <friction>
-            <torsional>
-              <coefficient>1.0</coefficient>
-              <surface_radius>0.0475</surface_radius>
-              <use_patch_radius>false</use_patch_radius>
-            </torsional>
-          </friction>
-        </surface>
-      </collision>
     </gazebo>
     <gazebo reference="caster_link_fl">
@@ -33,19 +20,6 @@
       <kp>1000000</kp>
       <kd>100</kd>
-      <mu1>100000.0</mu1>
-      <mu2>100000.0</mu2>
       <maxContacts>1</maxContacts>
       <minDepth>0.003</minDepth>
-      <collision name="wheel_link_fr_collision">
-        <surface>
-          <friction>
-            <torsional>
-              <coefficient>1.0</coefficient>
-              <surface_radius>0.0475</surface_radius>
-              <use_patch_radius>false</use_patch_radius>
-            </torsional>
-          </friction>
-        </surface>
-      </collision>
     </gazebo>
     <gazebo reference="caster_link_fr">
@@ -55,19 +29,6 @@
       <kp>1000000</kp>
       <kd>100</kd>
-      <mu1>100000.0</mu1>
-      <mu2>100000.0</mu2>
       <maxContacts>1</maxContacts>
       <minDepth>0.003</minDepth>
-      <collision name="wheel_link_bl_collision">
-        <surface>
-          <friction>
-            <torsional>
-              <coefficient>1.0</coefficient>
-              <surface_radius>0.0475</surface_radius>
-              <use_patch_radius>false</use_patch_radius>
-            </torsional>
-          </friction>
-        </surface>
-      </collision>
     </gazebo>
     <gazebo reference="caster_link_bl">
@@ -77,19 +38,6 @@
       <kp>1000000</kp>
       <kd>100</kd>
-      <mu1>100000.0</mu1>
-      <mu2>100000.0</mu2>
       <maxContacts>1</maxContacts>
       <minDepth>0.003</minDepth>
-      <collision name="wheel_link_br_collision">
-        <surface>
-          <friction>
-            <torsional>
-              <coefficient>1.0</coefficient>
-              <surface_radius>0.0475</surface_radius>
-              <use_patch_radius>false</use_patch_radius>
-            </torsional>
-          </friction>
-        </surface>
-      </collision>
     </gazebo>
     <gazebo reference="caster_link_br">

Commit message: Removed unnecessary file and corrected syntax.

File: urdf/youbot_base/base.gazebo.xacro (robot description, xacro)
@@ -4,5 +4,5 @@
        xmlns:interface="http://playerstage.sourceforge.net/gazebo/xmlschema/#interface"
        xmlns:xacro="http://www.ros.org/wiki/xacro">
-  <xacro:macro name="youbot_base_gazebo" params="namespace">
+  <xacro:macro name="youbot_base_gazebo">
     <gazebo reference="youbot_base">
     </gazebo>

File: urdf/youbot_base/base.urdf.xacro (robot description, xacro)
@@ -5,5 +5,4 @@
        xmlns:xacro="http://www.ros.org/wiki/xacro">
   <xacro:include filename="$(find youbot_description)/urdf/youbot_base/base.gazebo.xacro"/>
-  <xacro:include filename="$(find youbot_description)/urdf/youbot_base/base.transmission.xacro"/>
   <!-- simplified box collision geometry for base -->
   <xacro:property name="base_size_x" value="0.570"/>
@@ -11,8 +10,8 @@
   <xacro:property name="base_size_z" value="0.100"/>
   <xacro:property name="base_mass" value="22.0"/>
-  <property name="wheel_offset_x" value="0.228"  />
-  <property name="wheel_offset_y" value="0.158"  />
-  <property name="wheel_offset_z" value="-0.034" />
-  <xacro:property name="wheel_mass" value="1.4"/>
+  <xacro:property name="wheel_offset_x" value="0.228"  />
+  <xacro:property name="wheel_offset_y" value="0.158"  />
+  <xacro:property name="wheel_offset_z" value="-0.034" />
+  <xacro:property name="wheel_mass" value="0.4"/>
   <xacro:property name="wheel_radius" value="0.05"/>
   <xacro:property name="wheel_length" value="0.07"/>
@@ -185,6 +184,5 @@
     </link>
     <!-- extensions -->
-    <xacro:youbot_base_gazebo namespace="gazebo"/>
-    <xacro:youbot_base_transmission/>
+    <xacro:youbot_base_gazebo/>
   </xacro:macro>
 </robot>

File: urdf/youbot_gripper/gripper.urdf.xacro (robot description, xacro)
@@ -37,5 +37,5 @@
 		</link>
 		<joint name="${name}_finger_joint_l" type="prismatic">
-			<origin xyz="0.004 0.019 0.046" rpy="0 0 ${M_PI}" />
+			<origin xyz="0.004 0.015 0.046" rpy="0 0 ${M_PI}" />
 			<parent link="${name}_palm_link"/>
 			<child link="${name}_finger_link_l"/>
@@ -67,5 +67,5 @@
 		</link>
                <joint name="${name}_finger_joint_r" type="prismatic">
-			<origin xyz="0.004 -0.019 0.046" rpy="0 0 0" />
+			<origin xyz="0.004 -0.015 0.046" rpy="0 0 0" />
 			<parent link="${name}_palm_link"/>
 			<child link="${name}_finger_link_r"/>
