Commit message: Fixed inertia warning. Added friction to possibly fix gazebo robot slipping.

File: controller/ros_controller.urdf.xacro (robot description, xacro)
@@ -4,5 +4,8 @@
        xmlns:interface="http://playerstage.sourceforge.net/gazebo/xmlschema/#interface">
   <gazebo>
-    <plugin name="gazebo_ros_controller" filename="libgazebo_ros_control.so" />
+    <plugin name="gazebo_ros_controller" filename="libgazebo_ros_control.so">
+      <robotSimType>gazebo_ros_control/DefaultRobotHWSim</robotSimType>
+      <legacyModeNS>true</legacyModeNS>
+    </plugin>
   </gazebo>
 </robot>

File: urdf/sensors/intel_d435.gazebo.xacro (robot description, xacro)
@@ -6,4 +6,5 @@
   <xacro:macro name="intel_d435_gazebo" params="name">
     <gazebo reference="${name}_camera">
+      <material>Gazebo/Grey</material>
       <sensor type="depth" name="${name}_depth_frame_sensor">
         <always_on>true</always_on>
@@ -49,9 +50,9 @@
         <update_rate>20.0</update_rate>
         <camera>
-          <horizontal_fov>${69.4*M_PI/180.0}</horizontal_fov>
+          <horizontal_fov>${87.0*M_PI/180.0}</horizontal_fov>
           <image>
             <format>R8G8B8</format>
-            <width>1920</width>
-            <height>1080</height>
+            <width>1280</width>
+            <height>720</height>
           </image>
           <clip>

File: urdf/youbot_base/base.gazebo.xacro (robot description, xacro)
@@ -11,4 +11,19 @@
       <kp>1000000</kp>
       <kd>100</kd>
+      <mu1>100000.0</mu1>
+      <mu2>100000.0</mu2>
+      <maxContacts>1</maxContacts>
+      <minDepth>0.003</minDepth>
+      <collision name="wheel_link_fl_collision">
+        <surface>
+          <friction>
+            <torsional>
+              <coefficient>1.0</coefficient>
+              <surface_radius>0.0475</surface_radius>
+              <use_patch_radius>false</use_patch_radius>
+            </torsional>
+          </friction>
+        </surface>
+      </collision>
     </gazebo>
     <gazebo reference="caster_link_fl">
@@ -18,4 +33,19 @@
       <kp>1000000</kp>
       <kd>100</kd>
+      <mu1>100000.0</mu1>
+      <mu2>100000.0</mu2>
+      <maxContacts>1</maxContacts>
+      <minDepth>0.003</minDepth>
+      <collision name="wheel_link_fr_collision">
+        <surface>
+          <friction>
+            <torsional>
+              <coefficient>1.0</coefficient>
+              <surface_radius>0.0475</surface_radius>
+              <use_patch_radius>false</use_patch_radius>
+            </torsional>
+          </friction>
+        </surface>
+      </collision>
     </gazebo>
     <gazebo reference="caster_link_fr">
@@ -25,4 +55,19 @@
       <kp>1000000</kp>
       <kd>100</kd>
+      <mu1>100000.0</mu1>
+      <mu2>100000.0</mu2>
+      <maxContacts>1</maxContacts>
+      <minDepth>0.003</minDepth>
+      <collision name="wheel_link_bl_collision">
+        <surface>
+          <friction>
+            <torsional>
+              <coefficient>1.0</coefficient>
+              <surface_radius>0.0475</surface_radius>
+              <use_patch_radius>false</use_patch_radius>
+            </torsional>
+          </friction>
+        </surface>
+      </collision>
     </gazebo>
     <gazebo reference="caster_link_bl">
@@ -32,4 +77,19 @@
       <kp>1000000</kp>
       <kd>100</kd>
+      <mu1>100000.0</mu1>
+      <mu2>100000.0</mu2>
+      <maxContacts>1</maxContacts>
+      <minDepth>0.003</minDepth>
+      <collision name="wheel_link_br_collision">
+        <surface>
+          <friction>
+            <torsional>
+              <coefficient>1.0</coefficient>
+              <surface_radius>0.0475</surface_radius>
+              <use_patch_radius>false</use_patch_radius>
+            </torsional>
+          </friction>
+        </surface>
+      </collision>
     </gazebo>
     <gazebo reference="caster_link_br">

File: urdf/youbot_base/base.urdf.xacro (robot description, xacro)
@@ -33,9 +33,4 @@
   <xacro:macro name="youbot_base" params="name">
     <link name="${name}_footprint">
-      <inertial>
-        <mass value="0.1"/>
-        <origin xyz="0 0 ${-base_size_z / 2.0}" rpy="0 0 0"/>
-        <inertia ixx="1.0" ixy="0.0" ixz="0.0" iyy="1.0" iyz="0.0" izz="1.0"/>
-      </inertial>
       <visual>
         <origin xyz="0 0 0" rpy="0 0 0"/>
@@ -57,11 +52,4 @@
       <parent link="${name}_footprint"/>
     </joint>
-    <!-- Fix inertia warning
-    <link name="dummy"></link>
-    <joint name="dummy_joint" type="fixed">
-      <parent link="dummy"/>
-      <child link="base_footprint"/>
-    </joint>
-    Fix warning -->
     <link name="${name}_link">
       <inertial>
