Commit message: Updated origin of gripper. Updated values of release tolerance

File: urdf/youbot_gripper/grasp_fix_plugin.urdf.xacro (robot description, xacro)
@@ -21,5 +21,5 @@
                 <grip_count_threshold>4</grip_count_threshold>
                 <max_grip_count>8</max_grip_count>
-                <release_tolerance>0.005</release_tolerance>
+                <release_tolerance>0.0005</release_tolerance>
                 <disable_collisions_on_attach>false</disable_collisions_on_attach>
                 <contact_topic>__default_topic__</contact_topic>

File: urdf/youbot_gripper/gripper.urdf.xacro (robot description, xacro)
@@ -37,5 +37,5 @@
 		</link>
 		<joint name="${name}_finger_joint_l" type="prismatic">
-			<origin xyz="0.004 0.022 0.046" rpy="0 0 ${M_PI}" />
+			<origin xyz="0.004 0.024 0.046" rpy="0 0 ${M_PI}" />
 			<parent link="${name}_palm_link"/>
 			<child link="${name}_finger_link_l"/>
@@ -67,5 +67,5 @@
 		</link>
                <joint name="${name}_finger_joint_r" type="prismatic">
-			<origin xyz="0.004 -0.022 0.046" rpy="0 0 0" />
+			<origin xyz="0.004 -0.024 0.046" rpy="0 0 0" />
 			<parent link="${name}_palm_link"/>
 			<child link="${name}_finger_link_r"/>
