Commit message: Updated gripper file.

File: urdf/youbot_gripper/gripper.urdf.xacro (robot description, xacro)
@@ -36,5 +36,5 @@
 		</link>
 		<joint name="${name}_finger_joint_l" type="prismatic">
-			<origin xyz="0.004 0.008 0.046" rpy="0 0 ${M_PI}" />
+			<origin xyz="0.004 0.0205 0.046" rpy="0 0 ${M_PI}" />
 			<parent link="${name}_palm_link"/>
 			<child link="${name}_finger_link_l"/>
@@ -66,5 +66,5 @@
 		</link>
                <joint name="${name}_finger_joint_r" type="prismatic">
-			<origin xyz="0.004 -0.008 0.046" rpy="0 0 0" />
+			<origin xyz="0.004 -0.0205 0.046" rpy="0 0 0" />
 			<parent link="${name}_palm_link"/>
 			<child link="${name}_finger_link_r"/>

Commit message: Added backlash to z axis.

File: urdf/youbot_gripper/gripper.urdf.xacro (robot description, xacro)
@@ -37,5 +37,5 @@
 		</link>
 		<joint name="${name}_finger_joint_l" type="prismatic">
-			<origin xyz="0.004 0.024 0.046" rpy="0 0 ${M_PI}" />
+			<origin xyz="0.004 0.019 0.046" rpy="0 0 ${M_PI}" />
 			<parent link="${name}_palm_link"/>
 			<child link="${name}_finger_link_l"/>
@@ -67,5 +67,5 @@
 		</link>
                <joint name="${name}_finger_joint_r" type="prismatic">
-			<origin xyz="0.004 -0.024 0.046" rpy="0 0 0" />
+			<origin xyz="0.004 -0.019 0.046" rpy="0 0 0" />
 			<parent link="${name}_palm_link"/>
 			<child link="${name}_finger_link_r"/>
