Commit message: Fixed link4 and link5 friction accordingly to mas-group @4f4a865

File: urdf/youbot_arm/arm.urdf.xacro (robot description, xacro)
@@ -154,5 +154,5 @@
 			<axis xyz="0 1 0" />
 			<!--<calibration rising="${arm_4_ref}" falling="${arm_4_ref}"/>-->
-			<dynamics damping="1" friction="1" />
+			<dynamics damping="1" friction="0.5" />
 			<limit effort="${2.0}" velocity="${M_PI / 2.0}" lower="0" upper="${joint_4_limit}"/>
 			<!--safety_controller k_position="20" k_velocity="100" soft_lower_limit="0" soft_upper_limit="${joint_4_limit_soft}" /-->
@@ -186,5 +186,5 @@
 			<axis xyz="0 0 -1" />
 			<!--<calibration rising="${arm_5_ref}" falling="${arm_5_ref}"/>-->
-			<dynamics damping="1" friction="1" />
+			<dynamics damping="0.5" friction="0.5" />
 			<limit effort="${1.0}" velocity="${M_PI / 2.0}" lower="0" upper="${joint_5_limit}" />
       <!--safety_controller k_position="20" k_velocity="100" soft_lower_limit="0" soft_upper_limit="${joint_5_limit_soft}" /-->

Commit message: Added Grasp fix plugin to urdf (Link is in grasp fix plugin file). Updated Effort. Now the youbot can grab a bottle.

File: urdf/youbot_arm/arm.urdf.xacro (robot description, xacro)
@@ -155,5 +155,5 @@
 			<!--<calibration rising="${arm_4_ref}" falling="${arm_4_ref}"/>-->
 			<dynamics damping="1" friction="0.5" />
-			<limit effort="${2.0}" velocity="${M_PI / 2.0}" lower="0" upper="${joint_4_limit}"/>
+			<limit effort="${9.5}" velocity="${M_PI / 2.0}" lower="0" upper="${joint_4_limit}"/>
 			<!--safety_controller k_position="20" k_velocity="100" soft_lower_limit="0" soft_upper_limit="${joint_4_limit_soft}" /-->
 		</joint>

File: urdf/youbot_gripper/gripper.urdf.xacro (robot description, xacro)
@@ -6,4 +6,5 @@
 	<xacro:include filename="$(find youbot_description)/urdf/youbot_gripper/gripper.gazebo.xacro" />
 	<xacro:include filename="$(find youbot_description)/urdf/youbot_gripper/gripper.transmission.xacro" />
+	<xacro:include filename="$(find youbot_description)/urdf/youbot_gripper/grasp_fix_plugin.urdf.xacro" />
 	<xacro:include filename="$(find youbot_description)/urdf/youbot_gripper/limits.urdf.xacro" />
 	<xacro:macro name="youbot_gripper" params="parent name *origin">
@@ -36,5 +37,5 @@
 		</link>
 		<joint name="${name}_finger_joint_l" type="prismatic">
-			<origin xyz="0.004 0.0205 0.046" rpy="0 0 ${M_PI}" />
+			<origin xyz="0.004 0.022 0.046" rpy="0 0 ${M_PI}" />
 			<parent link="${name}_palm_link"/>
 			<child link="${name}_finger_link_l"/>
@@ -66,5 +67,5 @@
 		</link>
                <joint name="${name}_finger_joint_r" type="prismatic">
-			<origin xyz="0.004 -0.0205 0.046" rpy="0 0 0" />
+			<origin xyz="0.004 -0.022 0.046" rpy="0 0 0" />
 			<parent link="${name}_palm_link"/>
 			<child link="${name}_finger_link_r"/>
@@ -98,4 +99,5 @@
 		<xacro:youbot_gripper_gazebo name="${name}" />
 		<xacro:youbot_gripper_transmission name="${name}" />
+		<xacro:gzplugin_grasp_fix />
 	</xacro:macro>
 </robot>

Commit message: Updated effort value again

File: urdf/youbot_arm/arm.urdf.xacro (robot description, xacro)
@@ -155,5 +155,5 @@
 			<!--<calibration rising="${arm_4_ref}" falling="${arm_4_ref}"/>-->
 			<dynamics damping="1" friction="0.5" />
-			<limit effort="${9.5}" velocity="${M_PI / 2.0}" lower="0" upper="${joint_4_limit}"/>
+			<limit effort="${15.0}" velocity="${M_PI / 2.0}" lower="0" upper="${joint_4_limit}"/>
 			<!--safety_controller k_position="20" k_velocity="100" soft_lower_limit="0" soft_upper_limit="${joint_4_limit_soft}" /-->
 		</joint>

Commit message: More Force for joint 3 (from 6.0 Nm to 9.5 Nm).

File: urdf/youbot_arm/arm.urdf.xacro (robot description, xacro)
@@ -123,5 +123,5 @@
 			<axis xyz="0 1 0"/>
 			<dynamics damping="1" friction="0.5" />
-			<limit effort="${6.0}" velocity="${M_PI / 2.0}" lower="-${joint_3_limit}" upper="0"/>
+			<limit effort="${9.5}" velocity="${M_PI / 2.0}" lower="-${joint_3_limit}" upper="0"/>
       <!--safety_controller k_position="20" k_velocity="50" soft_lower_limit="-${joint_3_limit_soft}" soft_upper_limit="-${threshold}" /-->
 		</joint>
@@ -155,5 +155,5 @@
 			<!--<calibration rising="${arm_4_ref}" falling="${arm_4_ref}"/>-->
 			<dynamics damping="1" friction="0.5" />
-			<limit effort="${15.0}" velocity="${M_PI / 2.0}" lower="0" upper="${joint_4_limit}"/>
+			<limit effort="${9.5}" velocity="${M_PI / 2.0}" lower="0" upper="${joint_4_limit}"/>
 			<!--safety_controller k_position="20" k_velocity="100" soft_lower_limit="0" soft_upper_limit="${joint_4_limit_soft}" /-->
 		</joint>

Commit message: updated effort for arm link 1 and 2

File: urdf/youbot_arm/arm.urdf.xacro (robot description, xacro)
@@ -47,5 +47,5 @@
 			<!-- damping - N*s/m, N*s*m/rad -->
 			<!-- friction - N, N*m -->
-			<limit effort="${9.5}" velocity="${M_PI / 2.0}" lower="0" upper="${joint_1_limit}"/>
+			<limit effort="${14.0}" velocity="${M_PI / 2.0}" lower="0" upper="${joint_1_limit}"/>
 			<!--effort - N, N*m-->
 			<!--velocity - m/s, rad/s-->
@@ -84,5 +84,5 @@
 			<!--<calibration rising="${arm_2_ref}" falling="${arm_2_ref}"/>-->
 			<dynamics damping="1" friction="0.5" />
-			<limit effort="${9.5}" velocity="${M_PI / 2.0}" lower="0" upper="${joint_2_limit}"/>
+			<limit effort="${12.0}" velocity="${M_PI / 2.0}" lower="0" upper="${joint_2_limit}"/>
       <!--safety_controller k_position="20" k_velocity="${2*9.5/M_PI}" soft_lower_limit="${threshold}" soft_upper_limit="${joint_2_limit_soft}" /-->
 		</joint>

Commit message: Updated Descrption, Pick Server. New Routine Strategy. Updated Shakerbot Node.

File: urdf/youbot_arm/arm.urdf.xacro (robot description, xacro)
@@ -187,5 +187,5 @@
 			<!--<calibration rising="${arm_5_ref}" falling="${arm_5_ref}"/>-->
 			<dynamics damping="0.5" friction="0.5" />
-			<limit effort="${1.0}" velocity="${M_PI / 2.0}" lower="0" upper="${joint_5_limit}" />
+			<limit effort="${35.0}" velocity="${M_PI / 2.0}" lower="0" upper="${joint_5_limit}" />
       <!--safety_controller k_position="20" k_velocity="100" soft_lower_limit="0" soft_upper_limit="${joint_5_limit_soft}" /-->
 		</joint>

File: urdf/youbot_gripper/gripper.urdf.xacro (robot description, xacro)
@@ -8,4 +8,5 @@
 	<xacro:include filename="$(find youbot_description)/urdf/youbot_gripper/grasp_fix_plugin.urdf.xacro" />
 	<xacro:include filename="$(find youbot_description)/urdf/youbot_gripper/limits.urdf.xacro" />
+	<xacro:property name="finger_offset" value="0.025" />
 	<xacro:macro name="youbot_gripper" params="parent name *origin">
 		<!-- joint between arm_7_link and sdh_palm_link -->
@@ -37,5 +38,5 @@
 		</link>
 		<joint name="${name}_finger_joint_l" type="prismatic">
-			<origin xyz="0.004 0.015 0.046" rpy="0 0 ${M_PI}" />
+			<origin xyz="0.004 ${finger_offset} 0.046" rpy="0 0 ${M_PI}" />
 			<parent link="${name}_palm_link"/>
 			<child link="${name}_finger_link_l"/>
@@ -67,5 +68,5 @@
 		</link>
                <joint name="${name}_finger_joint_r" type="prismatic">
-			<origin xyz="0.004 -0.015 0.046" rpy="0 0 0" />
+			<origin xyz="0.004 -${finger_offset} 0.046" rpy="0 0 0" />
 			<parent link="${name}_palm_link"/>
 			<child link="${name}_finger_link_r"/>

Commit message: Updated grasp plugin values for better attaching and detaching. Update Torque for arm_link_5

File: urdf/youbot_arm/arm.urdf.xacro (robot description, xacro)
@@ -47,5 +47,5 @@
 			<!-- damping - N*s/m, N*s*m/rad -->
 			<!-- friction - N, N*m -->
-			<limit effort="${14.0}" velocity="${M_PI / 2.0}" lower="0" upper="${joint_1_limit}"/>
+			<limit effort="${35.0}" velocity="${M_PI / 2.0}" lower="0" upper="${joint_1_limit}"/>
 			<!--effort - N, N*m-->
 			<!--velocity - m/s, rad/s-->

File: urdf/youbot_gripper/grasp_fix_plugin.urdf.xacro (robot description, xacro)
@@ -19,7 +19,7 @@
                 <forces_angle_tolerance>100</forces_angle_tolerance>
                 <update_rate>4</update_rate>
-                <grip_count_threshold>4</grip_count_threshold>
-                <max_grip_count>8</max_grip_count>
-                <release_tolerance>0.0035</release_tolerance>
+                <grip_count_threshold>6</grip_count_threshold>
+                <max_grip_count>12</max_grip_count>
+                <release_tolerance>0.0028</release_tolerance>
                 <disable_collisions_on_attach>false</disable_collisions_on_attach>
                 <contact_topic>__default_topic__</contact_topic>

Commit message: Updated Bottleholder.stl. Updated Joint Force.

File: urdf/youbot_arm/arm.urdf.xacro (robot description, xacro)
@@ -84,5 +84,5 @@
 			<!--<calibration rising="${arm_2_ref}" falling="${arm_2_ref}"/>-->
 			<dynamics damping="1" friction="0.5" />
-			<limit effort="${12.0}" velocity="${M_PI / 2.0}" lower="0" upper="${joint_2_limit}"/>
+			<limit effort="${20.0}" velocity="${M_PI / 2.0}" lower="0" upper="${joint_2_limit}"/>
       <!--safety_controller k_position="20" k_velocity="${2*9.5/M_PI}" soft_lower_limit="${threshold}" soft_upper_limit="${joint_2_limit_soft}" /-->
 		</joint>
@@ -123,5 +123,5 @@
 			<axis xyz="0 1 0"/>
 			<dynamics damping="1" friction="0.5" />
-			<limit effort="${9.5}" velocity="${M_PI / 2.0}" lower="-${joint_3_limit}" upper="0"/>
+			<limit effort="${20.0}" velocity="${M_PI / 2.0}" lower="-${joint_3_limit}" upper="0"/>
       <!--safety_controller k_position="20" k_velocity="50" soft_lower_limit="-${joint_3_limit_soft}" soft_upper_limit="-${threshold}" /-->
 		</joint>

File: urdf/youbot_plate/plate.urdf.xacro (robot description, xacro)
@@ -42,14 +42,14 @@
 			</inertial>
 			<visual>
-				<origin xyz="-0.05 0.095 0.0225" rpy="${M_PI/2} 0 0" />
+				<origin xyz="-0.05 0.095 0.0225" rpy="0 0 0" />
 				<geometry>
-					<mesh filename="package://youbot_description/meshes/bottleholder.stl" scale="0.001 0.001 0.001"/>
+					<mesh filename="package://youbot_description/meshes/bottleholder_new.stl" /> <!-- scale="0.001 0.001 0.001"/>-->
 				</geometry>
 				<material name="DarkGrey"/>
 			</visual>
 			<collision>
-				<origin xyz="-0.05 0.095 0.0225" rpy="${M_PI/2} 0 0" />
+				<origin xyz="-0.05 0.095 0.0225" rpy="0 0 0" />
 				<geometry>
-					<mesh filename="package://youbot_description/meshes/bottleholder.stl" scale="0.001 0.001 0.001"/>
+					<mesh filename="package://youbot_description/meshes/bottleholder_new.stl" /> <!--scale="0.001 0.001 0.001"/>-->
 				</geometry>
 			</collision>
